File: LED Chaser/LED Chaser.sch (KiCad schematic (older format))
At the start: 20 parts, among them J1 power in, U1 NE555D, U2 4017

Commit message: added power supply
Parts:
- added C3: 27uF, Capacitor_SMD:CP_Elec_6.3x7.7, symbol Device:CP1
- added C4: 1nF, Capacitor_SMD:C_0805_2012Metric, symbol Device:C
- added C5: 470uF, Capacitor_SMD:CP_Elec_6.3x7.7, symbol Device:CP1
- added D12: D_Zener, Diode_SMD:D_0805_2012Metric, symbol Device:D_Zener
- added L1: 33uH, Inductor_SMD:L_Bourns_SRR1260, symbol Device:L
- added R4: 1k, Resistor_SMD:R_0805_2012Metric, symbol Device:R
- added R5: 3.83k, Resistor_SMD:R_0805_2012Metric, symbol Device:R
- added U3: LM2596S-ADJ, Package_TO_SOT_SMD:TO-263-5_TabPin3, symbol Regulator_Switching:LM2596S-ADJ
- C1: value C -> 0.01uF
- C2: value C -> 10uF
- R1: value R -> 10k
- R2, R3: value R -> 680R
- RV1: value R_POT -> 10k
Connections:
- net GND: now also C3.2, C5.2, D12.2 (A), R4.1, U3.3 (GND)
- net VCC: now also C4.1, C5.1, L1.2, R5.1; no longer J1.2 (Pin_2)
- new net: C3.1, J1.2 (Pin_2), U3.1 (VIN)
- new net: D12.1 (K), L1.1, U3.2 (OUT)
- new net: C4.2, R4.2, R5.2, U3.4 (FB)
- no-connect marks 1 -> 2
Other:
- note added: "4017 Decade counter"
- note added: "555 Timer"
- note added: "LEDs"
- note added: "Power Supply"
- moved on the sheet: C1, C2, D1, D10, D11, D2, D3, D4, D5, D6, D7, D8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
